File: PCBs/MOL-v1.sch (EAGLE design)
At the start: 25 parts, among them IC1 ULN2803, IC2 ULN2803, U1 SN74LVC2G04DBV, U2 JOYSTICKPTH, U3 JOYSTICKPTH

Commit message: initial version of MOL pcb schematic
Other:
- note added: "I2C"
- note added: "TEENSY 3.6"
- moved on the sheet: J1, J2, J_REG_5V_1, MOTORS1, POWER-5V, U1, U2, U3
