File: PCBs/MOL-v1.sch (EAGLE design)
At the start: 27 parts, among them IC1 ULN2803, IC2 ULN2803, U1 SN74LVC2G04DBV, U2 JOYSTICKPTH, U3 JOYSTICKPTH

Commit message: using git for real
Parts:
- removed BUTTON1: DTS-6, switch-tact:DTS-6
- removed J_REG_5V_1: POLOLU_VOLTAGE_REGULATORS_3PIN, CMU-ArtFab:POLOLU_VOLTAGE_REGULATORS_3PIN
- removed KNOB1: (no value), CMU-ArtFab:POT
- removed LED1: (no value), led:LED3MM
- added GND-SHRT, VIN, VOUT: (no value), CMU-ArtFab:M02LOCK
- added R10, R11, R12, R17, R18, R19, R2, R20, R3, R4, R5, R6, R9: (no value), SparkFun-Resistors:RESISTOREZ
- added S10, S11, S12, S3, S4, S5, S6, S7, S8, S9: SW-LEDPTH, Daniel:SW-LEDPTH
- added TM1, TM10, TM11, TM12, TM2, TM3, TM4, TM5, TM6, TM7, TM8, TM9: (no value), Daniel:TRIM
- J1: value (none) -> SERVO 1
- J2: value (none) -> SERVO 2
- R1, R13, R14, R15, R16: device CMU-ArtFab:R-US_R0603 -> SparkFun-Resistors:RESISTOREZ
Connections:
- removed net KNOB1: KNOB1.WIPER
- removed net VCC: KNOB1.IN
- new net N$10: R4.1, S4.A
- new net N$15: R9.1, S9.A
- new net N$16: R10.1, S10.A
- new net N$17: R11.1, S11.A
- new net N$18: R12.1, S12.A
- new net N$19: R17.1, S5.A
- new net N$20: R18.1, S6.A
- new net N$21: R19.1, S7.A
- new net N$22: R20.1, S8.A
- new net N$8: R2.1, S2.A
- new net N$9: R3.1, S3.A
- net +3V3: now also TM1.A, TM10.A, TM11.A, TM12.A, TM2.A, TM3.A, TM4.A, TM5.A, TM6.A, TM7.A, TM8.A, TM9.A
- net +5V: now also R5.1, R6.1, VIN.1; no longer J_REG_5V_1.VIN
- net A1: now also TM1.S, U$1.14/A0/PWM/ALT-SCK0; no longer U$1.33/A14/CAN1TX/TX5/ALT-SCL0
- net A10: now also TM10.S, U$1.DAC1; no longer U$1.14/A0/PWM/ALT-SCK0
- net A11: now also TM11.S, U$1.A10; no longer U$1.15/A1/CS0-4/T
- net A12: now also TM12.S, U$1.A11; no longer U$1.16/A2/PWM/T/ALT-SCL0
- net A2: now also TM2.S, U$1.15/A1/CS0-4/T; no longer U$1.34/A15/CAN1RX/RX5/ALT-SDA0
- net A3: now also TM3.S, U$1.16/A2/PWM/T/ALT-SCL0; no longer U$1.35/A16/PWM
- net A4: now also TM4.S, U$1.33/A14/CAN1TX/TX5/ALT-SCL0; no longer U$1.36/A17/PWM
- net A5: now also TM5.S, U$1.34/A15/CAN1RX/RX5/ALT-SDA0; no longer U$1.39/A20/ALT-MISO0
- net A6: now also TM6.S, U$1.35/A16/PWM; no longer U$1.DAC0
- net A7: now also TM7.S, U$1.36/A17/PWM; no longer U$1.DAC1
- net A8: now also TM8.S, U$1.39/A20/ALT-MISO0; no longer U$1.A10
- net A9: now also TM9.S, U$1.DAC0; no longer U$1.A11
- net AGND: now also TM1.E, TM10.E, TM11.E, TM12.E, TM2.E, TM3.E, TM4.E, TM5.E, TM6.E, TM7.E, TM8.E, TM9.E; no longer KNOB1.OUT
- net B1: now also S1.3; no longer BUTTON1.3
- net B10: now also S10.3
- net B11: now also S11.3
- net B12: now also S12.3
- net B2: now also S2.3
- net B3: now also S3.3
- net B4: now also S4.3
- net B5: now also S5.3
- net B6: now also S6.3
- net B7: now also S7.3
- net B8: now also S8.3
- net B9: now also S9.3
- net GND: now also GND-SHRT.2, S1.1, S1.C, S10.1, S10.C, S11.1, S11.C, S12.1, S12.C, S2.1, S2.C, S3.1, S3.C, S4.1, S4.C, S5.1, S5.C, S6.1, S6.C, S7.1, S7.C, S8.1, S8.C, S9.1, S9.C, VIN.2, VOUT.1; no longer BUTTON1.1, J_REG_5V_1.GND, LED1.C
- net GND_MOT: now also GND-SHRT.1
- net I2C_SCL: now also R5.2
- net I2C_SDA: now also R6.2
- net LED10: now also R10.2
- net LED11: now also R11.2
- net LED12: now also R12.2
- net LED2: now also R2.2
- net LED3: now also R3.2
- net LED4: now also R4.2
- net LED5: now also R17.2
- net LED6: now also R18.2
- net LED7: now also R19.2
- net LED8: now also R20.2
- net LED9: now also R9.2
- net N$1: now also S1.A; no longer LED1.A
- net S1: no longer J2.3
- net S2: now also J2.3
- net VMOT: now also VOUT.2; no longer J_REG_5V_1.VOUT
Other:
- note removed: "***Part needs to change to our knobs http://www.taydaelectronics.com/10k-ohm-linear-taper-potentiometer-round-shaft-pcb-9mm.html"
- moved on the sheet: I2C-0, IC1, IC2, J1, J2, LED13, LED14, LED15, LED16, MOTORS1, POWER-5V, R1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
