File: PCBs/MOL-v1.sch (EAGLE design)
At the start: 61 parts, among them IC1 ULN2803, IC2 ULN2803, J1 SERVO 1, J2 SERVO 2, U1 SN74LVC2G04DBV, U2 JOYSTICKPTH, U3 JOYSTICKPTH

Commit message: breakouts
Parts:
- added J3, J4, J5, J6, J7, J8: (no value), SparkFun-Connectors:M031X03_NO_SILK
Connections:
- net +3V3: now also J3.1, J4.1, J5.1, J6.1, J7.1, J8.1
- net A1: now also J3.2
- net A10: now also J8.2
- net A2: now also J4.2
- net A5: now also J5.2
- net A6: now also J6.2
- net A9: now also J7.2
- net AGND: now also J3.3, J4.3, J5.3, J6.3, J7.3, J8.3
Changed lines of the file:
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@@
 <part name="VIN" library="CMU-ArtFab" deviceset="M02" device="LOCK"/>
 <part name="VOUT" library="CMU-ArtFab" deviceset="M02" device="LOCK"/>
+<part name="J3" library="SparkFun-Connectors" deviceset="M03" device="1X03_NO_SILK"/>
+<part name="J4" library="SparkFun-Connectors" deviceset="M03" device="1X03_NO_SILK"/>
+<part name="J5" library="SparkFun-Connectors" deviceset="M03" device="1X03_NO_SILK"/>
+<part name="J6" library="SparkFun-Connectors" deviceset="M03" device="1X03_NO_SILK"/>
+<part name="J7" library="SparkFun-Connectors" deviceset="M03" device="1X03_NO_SILK"/>
+<part name="J8" library="SparkFun-Connectors" deviceset="M03" device="1X03_NO_SILK"/>
 </parts>
 <sheets>
@@
 Digikey: 563-1933-ND
 Cheaper than sparkfun, LED color is variable, and uses less current</text>
-<wire x1="-99.06" y1="-40.64" x2="-43.18" y2="-40.64" width="0.1524" layer="90"/>
+<wire x1="-101.6" y1="-40.64" x2="-43.18" y2="-40.64" width="0.1524" layer="90"/>
 <wire x1="-43.18" y1="-40.64" x2="170.18" y2="-40.64" width="0.1524" layer="90"/>
 <wire x1="170.18" y1="-40.64" x2="170.18" y2="-152.4" width="0.1524" layer="90"/>
-<wire x1="170.18" y1="-152.4" x2="-99.06" y2="-152.4" width="0.1524" layer="90"/>
-<wire x1="-99.06" y1="-152.4" x2="-99.06" y2="-40.64" width="0.1524" layer="90"/>
+<wire x1="170.18" y1="-152.4" x2="-101.6" y2="-152.4" width="0.1524" layer="90"/>
+<wire x1="-101.6" y1="-152.4" x2="-101.6" y2="-40.64" width="0.1524" layer="90"/>
 <text x="-101.6" y="22.86" size="6.4516" layer="91">KNOB+LED+BUTTON
 (we need 12 of these)</text>
@@
 <instance part="VIN" gate="G$1" x="233.68" y="86.36" rot="R180"/>
 <instance part="VOUT" gate="G$1" x="248.92" y="83.82"/>
+<instance part="J3" gate="G$1" x="-160.02" y="-81.28"/>
+<instance part="J4" gate="G$1" x="-160.02" y="-96.52"/>
+<instance part="J5" gate="G$1" x="-160.02" y="-111.76"/>
+<instance part="J6" gate="G$1" x="-132.08" y="-81.28"/>
+<instance part="J7" gate="G$1" x="-132.08" y="-96.52"/>
+<instance part="J8" gate="G$1" x="-132.08" y="-111.76"/>
 </instances>
 <busses>
@@
 <wire x1="139.7" y1="-142.24" x2="139.7" y2="-144.78" width="0.1524" layer="91"/>
 </segment>
+<segment>
+<pinref part="J3" gate="G$1" pin="3"/>
+<wire x1="-152.4" y1="-78.74" x2="-144.78" y2="-78.74" width="0.1524" layer="91"/>
+<label x="-144.78" y="-78.74" size="1.016" layer="95" xref="yes"/>
+</segment>
+<segment>
+<pinref part="J4" gate="G$1" pin="3"/>
+<wire x1="-152.4" y1="-93.98" x2="-144.78" y2="-93.98" width="0.1524" layer="91"/>
+<label x="-144.78" y="-93.98" size="1.016" layer="95" xref="yes"/>
+</segment>
+<segment>
+<pinref part="J5" gate="G$1" pin="3"/>
+<wire x1="-152.4" y1="-109.22" x2="-144.78" y2="-109.22" width="0.1524" layer="91"/>
+<label x="-144.78" y="-109.22" size="1.016" layer="95" xref="yes"/>
+</segment>
+<segment>
+<pinref part="J6" gate="G$1" pin="3"/>
+<wire x1="-124.46" y1="-78.74" x2="-116.84" y2="-78.74" width="0.1524" layer="91"/>
+<label x="-116.84" y="-78.74" size="1.016" layer="95" xref="yes"/>
+</segment>
+<segment>
+<pinref part="J7" gate="G$1" pin="3"/>
+<wire x1="-124.46" y1="-93.98" x2="-116.84" y2="-93.98" width="0.1524" layer="91"/>
+<label x="-116.84" y="-93.98" size="1.016" layer="95" xref="yes"/>
+</segment>
+<segment>
+<pinref part="J8" gate="G$1" pin="3"/>
+<wire x1="-124.46" y1="-109.22" x2="-116.84" y2="-109.22" width="0.1524" layer="91"/>
+<label x="-116.84" y="-109.22" size="1.016" layer="95" xref="yes"/>
+</segment>
 </net>
 <net name="L1" class="0">
@@
 <label x="-78.74" y="157.48" size="1.016" layer="95" rot="R180" xref="yes"/>
 </segment>
+<segment>
+<pinref part="J3" gate="G$1" pin="2"/>
+<wire x1="-152.4" y1="-81.28" x2="-144.78" y2="-81.28" width="0.1524" layer="91"/>
+<label x="-144.78" y="-81.28" size="1.016" layer="95" xref="yes"/>
+</segment>
 </net>
 <net name="A2" class="3">
@@
 <label x="-78.74" y="154.94" size="1.016" layer="95" rot="R180" xref="yes"/>
 </segment>
+<segment>
+<pinref part="J4" gate="G$1" pin="2"/>
+<wire x1="-152.4" y1="-96.52" x2="-144.78" y2="-96.52" width="0.1524" layer="91"/>
+<label x="-144.78" y="-96.52" size="1.016" layer="95" xref="yes"/>
+</segment>
 </net>
 <net name="A3" class="3">
@@
 <label x="-78.74" y="106.68" size="1.016" layer="95" rot="R180" xref="yes"/>
 </segment>
+<segment>
+<pinref part="J5" gate="G$1" pin="2"/>
+<wire x1="-152.4" y1="-111.76" x2="-144.78" y2="-111.76" width="0.1524" layer="91"/>
+<label x="-144.78" y="-111.76" size="1.016" layer="95" xref="yes"/>
+</segment>
 </net>
 <net name="A6" class="3">
@@
 <label x="-78.74" y="104.14" size="1.016" layer="95" rot="R180" xref="yes"/>
 </segment>
+<segment>
+<pinref part="J6" gate="G$1" pin="2"/>
+<wire x1="-124.46" y1="-81.28" x2="-116.84" y2="-81.28" width="0.1524" layer="91"/>
+<label x="-116.84" y="-81.28" size="1.016" layer="95" xref="yes"/>
+</segment>
 </net>
 <net name="A7" class="3">
@@
 <wire x1="-5.08" y1="157.48" x2="0" y2="157.48" width="0.1524" layer="91"/>
 <label x="0" y="157.48" size="1.016" layer="95" xref="yes"/>
+</segment>
+<segment>
+<pinref part="J8" gate="G$1" pin="2"/>
+<wire x1="-124.46" y1="-111.76" x2="-116.84" y2="-111.76" width="0.1524" layer="91"/>
+<label x="-116.84" y="-111.76" size="1.016" layer="95" xref="yes"/>
 </segment>
 </net>
@@
 <label x="0" y="154.94" size="1.016" layer="95" xref="yes"/>
 </segment>
+<segment>
+<pinref part="J7" gate="G$1" pin="2"/>
+<wire x1="-124.46" y1="-96.52" x2="-116.84" y2="-96.52" width="0.1524" layer="91"/>
+<label x="-116.84" y="-96.52" size="1.016" layer="95" xref="yes"/>
+</segment>
 </net>
 <net name="N$2" class="0">
@@
 <label x="139.7" y="-124.46" size="1.016" layer="95" rot="R180" xref="yes"/>
 </segment>
-</net>
+<segment>
+<pinref part="J3" gate="G$1" pin="1"/>
+<wire x1="-152.4" y1="-83.82" x2="-144.78" y2="-83.82" width="0.1524" layer="91"/>
+<label x="-144.78" y="-83.82" size="1.016" layer="95" xref="yes"/>
+</segment>
+<segment>
+<pinref part="J4" gate="G$1" pin="1"/>
+<wire x1="-152.4" y1="-99.06" x2="-144.78" y2="-99.06" width="0.1524" layer="91"/>
+<label x="-144.78" y="-99.06" size="1.016" layer="95" xref="yes"/>
+</segment>
+<segment>
+<pinref part="J5" gate="G$1" pin="1"/>
+<wire x1="-152.4" y1="-114.3" x2="-144.78" y2="-114.3" width="0.1524" layer="91"/>
+<label x="-144.78" y="-114.3" size="1.016" layer="95" xref="yes"/>
+</segment>
+<segment>
+<pinref part="J6" gate="G$1" pin="1"/>
+<wire x1="-124.46" y1="-83.82" x2="-116.84" y2="-83.82" width="0.1524" layer="91"/>
+<label x="-116.84" y="-83.82" size="1.016" layer="95" xref="yes"/>
+</segment>
+<segment>
+<pinref part="J7" gate="G$1" pin="1"/>
+<wire x1="-124.46" y1="-99.06" x2="-116.84" y2="-99.06" width="0.1524" layer="91"/>
+<label x="-116.84" y="-99.06" size="1.016" layer="95" xref="yes"/>
+</segment>
+<segment>
+<pinref part="J8" gate="G$1" pin="1"/>
+<wire x1="-124.46" y1="-114.3" x2="-116.84" y2="-114.3" width="0.1524" layer="91"/>
+<label x="-116.84" y="-114.3" size="1.016" layer="95" xref="yes"/>
+</segment>
+</net>
