File: PCBs/MOL-v1.2.brd (EAGLE design)
At the start: 252.7 x 75.9 mm, 27 parts, among them IC1 ULN2803, IC2 ULN2803, U1 SN74LVC2G04DBV, U2 JOYSTICKPTH, U3 JOYSTICKPTH

Commit message: my stuff
Parts:
- removed BUTTON1: DTS-6, switch-tact:DTS-6
- removed KNOB1: (no value), CMU-ArtFab:ALPS_POT
- removed LED1: (no value), led:LED3MM
- added R2, R3, R4: (no value), CMU-ArtFab:R0603
- added S3, S4: SW-LEDPTH, Daniel:TR2-SWITCH-MOMENTARY-LED
- added TM1, TM2, TM3, TM4: (no value), Daniel:TRIM-PCB-9MM
- moved S2 487.9 mm to (99.7, 39.1)
- moved R1 99.7 mm to (99.7, 21.0)
- moved S1 91.4 mm to (111.1, 39.1)
- moved MOTORS1 24.1 mm to (52.1, -80.0)
- moved U$1 5.08 mm to (19.1, 17.8)
Connections:
- removed net KNOB1: KNOB1.P$2
- new net N$10: R4.1, S4.A
- new net N$8: R2.1, S2.A
- new net N$9: R3.1, S3.A
- net A1: now also TM1.2
- net A2: now also TM2.2
- net A3: now also TM3.2
- net A4: now also TM4.2
- net AGND: now also TM1.3, TM2.3, TM3.3, TM4.3; no longer KNOB1.P$1
- net B1: now also S1.3; no longer BUTTON1.3
- net B2: now also S2.3
- net B3: now also S3.3
- net B4: now also S4.3
- net GND: now also S1.1, S1.C, S2.1, S2.C, S3.1, S3.C, S4.1, S4.C; no longer BUTTON1.1, LED1.K
- net L1: now also R1.2
- net L2: now also R2.2
- net L3: now also R3.2
- net L4: now also R4.2
- net LED1: no longer R1.2
- net N$1: now also S1.A; no longer LED1.A
- net VCC: now also TM1.1, TM2.1, TM3.1, TM4.1, U$1.5V; no longer KNOB1.P$3
