File: PCBs/MOL-v1.2.sch (EAGLE design)
At the start: 27 parts, among them IC1 ULN2803, IC2 ULN2803, U1 SN74LVC2G04DBV, U2 JOYSTICKPTH, U3 JOYSTICKPTH

Commit message: my stuff
Parts:
- removed BUTTON1: DTS-6, switch-tact:DTS-6
- removed KNOB1: (no value), CMU-ArtFab:POT
- removed LED1: (no value), led:LED3MM
- added R2, R3, R4: (no value), CMU-ArtFab:R-US_R0603
- added S3, S4: SW-LEDPTH, Daniel:SW-LEDPTH
- added TM1, TM2, TM3, TM4: (no value), Daniel:TRIM
Connections:
- removed net KNOB1: KNOB1.WIPER
- new net N$10: R4.1, S4.A
- new net N$8: R2.1, S2.A
- new net N$9: R3.1, S3.A
- net A1: now also TM1.S
- net A2: now also TM2.S
- net A3: now also TM3.S
- net A4: now also TM4.S
- net AGND: now also TM1.E, TM2.E, TM3.E, TM4.E; no longer KNOB1.OUT
- net B1: now also S1.3; no longer BUTTON1.3
- net B2: now also S2.3
- net B3: now also S3.3
- net B4: now also S4.3
- net GND: now also S1.1, S1.C, S2.1, S2.C, S3.1, S3.C, S4.1, S4.C; no longer BUTTON1.1, LED1.C
- net L1: now also R1.2
- net L2: now also R2.2
- net L3: now also R3.2
- net L4: now also R4.2
- net LED1: no longer R1.2
- net N$1: now also S1.A; no longer LED1.A
- net VCC: now also TM1.A, TM2.A, TM3.A, TM4.A, U$1.5V; no longer KNOB1.IN
Other:
- note removed: "***Part needs to change to our knobs http://www.taydaelectronics.com/10k-ohm-linear-taper-potentiometer-round-shaft-pcb-9mm.html"
- moved on the sheet: R1, S1, S2
