File: PCBs/MOL-v1.2b.brd (EAGLE design)
At the start: 252.7 x 75.9 mm, 27 parts, among them IC1 ULN2803, IC2 ULN2803, U1 SN74LVC2G04DBV, U2 JOYSTICKPTH, U3 JOYSTICKPTH

Commit message: my stuff
Parts:
- removed BUTTON1: DTS-6, switch-tact:DTS-6
- removed KNOB1: (no value), CMU-ArtFab:ALPS_POT
- removed LED1: (no value), led:LED3MM
- added R2, R3, R4: (no value), CMU-ArtFab:R0603
- added S3, S4: SW-LEDPTH, Daniel:TR2-SWITCH-MOMENTARY-LED
- added TM1, TM2, TM3, TM4: (no value), Daniel:TRIM-PCB-9MM
- moved S2 487.9 mm to (99.7, 39.1)
- moved R16 440.3 mm to (31.8, 62.2)
- moved LED16 435.2 mm to (31.8, 68.6)
- moved R15 421.6 mm to (22.9, 62.2)
- moved LED15 419.7 mm to (22.9, 68.6)
- moved R14 404.2 mm to (14.0, 62.2)
- moved LED14 399.3 mm to (14.0, 68.6)
- moved I2C-0 395.1 mm to (12.7, 10.2)
- moved R13 384.1 mm to (6.35, 62.2)
- moved LED13 379.2 mm to (6.35, 68.6)
- moved IC2 347.0 mm to (128.3, 10.2)
- moved U3 330.0 mm to (156.2, 24.1)
- moved J_REG_5V_1 322.1 mm to (196.8, 20.3)
- moved IC1 312.0 mm to (97.8, 8.89)
- moved U2 292.9 mm to (175.3, 55.9)
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Connections:
- removed net KNOB1: KNOB1.P$2
- new net N$10: R4.1, S4.A
- new net N$8: R2.1, S2.A
- new net N$9: R3.1, S3.A
- net A1: now also TM1.2
- net A2: now also TM2.2
- net A3: now also TM3.2
- net A4: now also TM4.2
- net AGND: now also TM1.3, TM2.3, TM3.3, TM4.3; no longer KNOB1.P$1
- net B1: now also S1.3; no longer BUTTON1.3
- net B2: now also S2.3
- net B3: now also S3.3
- net B4: now also S4.3
- net GND: now also S1.1, S1.C, S2.1, S2.C, S3.1, S3.C, S4.1, S4.C; no longer BUTTON1.1, LED1.K
- net L1: now also R1.2
- net L2: now also R2.2
- net L3: now also R3.2
- net L4: now also R4.2
- net LED1: no longer R1.2
- net N$1: now also S1.A; no longer LED1.A
- net VCC: now also TM1.1, TM2.1, TM3.1, TM4.1, U$1.5V; no longer KNOB1.P$3
Routing:
- net GND: track 0.00 -> 472.4 mm, vias 0 -> 2
- net +3V3: track 0.00 -> 372.7 mm, vias 0 -> 2
- net AGND: track 0.00 -> 334.7 mm
- net +5V: track 0.00 -> 274.8 mm, vias 0 -> 1
- net M_PWMA: track 0.00 -> 242.9 mm
- net M_PWMB: track 0.00 -> 222.3 mm
- net M_AIN: track 0.00 -> 220.7 mm
- net M_BIN: track 0.00 -> 215.1 mm
- net S_JOYB: track 0.00 -> 198.2 mm
- net S_JOYH: track 0.00 -> 178.1 mm
- net M_JOYB: track 0.00 -> 175.4 mm
- net M_JOYH: track 0.00 -> 169.9 mm, vias 0 -> 1
- net M_JOYV: track 0.00 -> 159.1 mm, vias 0 -> 2
- net L2: track 0.00 -> 147.3 mm, vias 0 -> 1
- net L3: track 0.00 -> 146.6 mm, vias 0 -> 1
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