File: PCBs/MOL-v1.3.sch (EAGLE design)
At the start: 27 parts, among them IC1 ULN2803, IC2 ULN2803, U1 SN74LVC2G04DBV, U2 JOYSTICKPTH, U3 JOYSTICKPTH

Commit message: my stuff
Parts:
- removed BUTTON1: DTS-6, switch-tact:DTS-6
- removed KNOB1: (no value), CMU-ArtFab:POT
- removed LED1: (no value), led:LED3MM
- added R10, R11, R12, R17, R18, R19, R2, R20, R3, R4, R9: (no value), CMU-ArtFab:R-US_R0603
- added S10, S11, S12, S13, S14, S15, S16, S3, S4, S9: SW-LEDPTH, Daniel:SW-LEDPTH
- added TM1, TM10, TM11, TM12, TM13, TM14, TM15, TM16, TM2, TM3, TM4, TM9: (no value), Daniel:TRIM
Connections:
- removed net KNOB1: KNOB1.WIPER
- new net N$10: R4.1, S4.A
- new net N$15: R9.1, S9.A
- new net N$16: R10.1, S10.A
- new net N$17: R11.1, S11.A
- new net N$18: R12.1, S12.A
- new net N$19: R17.1, S13.A
- new net N$20: R18.1, S14.A
- new net N$21: R19.1, S15.A
- new net N$22: R20.1, S16.A
- new net N$8: R2.1, S2.A
- new net N$9: R3.1, S3.A
- net A1: now also TM1.S
- net A10: now also TM10.S
- net A11: now also TM11.S
- net A12: now also TM12.S
- net A2: now also TM2.S
- net A3: now also TM3.S
- net A4: now also TM4.S
- net A5: now also TM13.S
- net A6: now also TM14.S
- net A7: now also TM15.S
- net A8: now also TM16.S
- net A9: now also TM9.S
- net AGND: now also TM1.E, TM10.E, TM11.E, TM12.E, TM13.E, TM14.E, TM15.E, TM16.E, TM2.E, TM3.E, TM4.E, TM9.E; no longer KNOB1.OUT
- net B1: now also S1.3; no longer BUTTON1.3
- net B10: now also S10.3
- net B11: now also S11.3
- net B12: now also S12.3
- net B2: now also S2.3
- net B3: now also S3.3
- net B4: now also S4.3
- net B5: now also S13.3
- net B6: now also S14.3
- net B7: now also S15.3
- net B8: now also S16.3
- net B9: now also S9.3
- net GND: now also S1.1, S1.C, S10.1, S10.C, S11.1, S11.C, S12.1, S12.C, S13.1, S13.C, S14.1, S14.C, S15.1, S15.C, S16.1, S16.C, S2.1, S2.C, S3.1, S3.C, S4.1, S4.C, S9.1, S9.C; no longer BUTTON1.1, LED1.C
- net L1: now also R1.2
- net L10: now also R10.2
- net L11: now also R11.2
- net L12: now also R12.2
- net L2: now also R2.2
- net L3: now also R3.2
- net L4: now also R4.2
- net L5: now also R17.2
- net L6: now also R18.2
- net L7: now also R19.2
- net L8: now also R20.2
- net L9: now also R9.2
- net LED1: no longer R1.2
- net N$1: now also S1.A; no longer LED1.A
- net VCC: now also TM1.A, TM10.A, TM11.A, TM12.A, TM13.A, TM14.A, TM15.A, TM16.A, TM2.A, TM3.A, TM4.A, TM9.A, U$1.5V; no longer KNOB1.IN
Other:
- note removed: "***Part needs to change to our knobs http://www.taydaelectronics.com/10k-ohm-linear-taper-potentiometer-round-shaft-pcb-9mm.html"
- moved on the sheet: I2C-0, IC1, IC2, J1, J2, J_REG_5V_1, LED13, LED14, LED15, LED16, MOTORS1, POWER-5V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
