File: PCBs/MOL-v1.4.brd (EAGLE design)
At the start: 252.7 x 75.9 mm, 27 parts, among them IC1 ULN2803, IC2 ULN2803, U1 SN74LVC2G04DBV, U2 JOYSTICKPTH, U3 JOYSTICKPTH

Commit message: my stuff
Parts:
- removed BUTTON1: DTS-6, switch-tact:DTS-6
- removed J_REG_5V_1: POLOLU_VOLTAGE_REGULATORS_3PIN, CMU-ArtFab:POLOLU_5V-12V_STEPUP_U3V12F5-U3V12F12
- removed KNOB1: (no value), CMU-ArtFab:ALPS_POT
- removed LED1: (no value), led:LED3MM
- added R10, R11, R12, R17, R18, R19, R2, R20, R3, R4, R5, R6, R9: (no value), CMU-ArtFab:R0603
- added REG1: BUCK-CONVERTER, Daniel:BUCK-CONVERTER
- added S10, S11, S12, S13, S14, S15, S16, S3, S4, S9: SW-LEDPTH, Daniel:TR2-SWITCH-MOMENTARY-LED
- added TM1, TM10, TM11, TM12, TM13, TM14, TM15, TM16, TM2, TM3, TM4, TM9: (no value), Daniel:TRIM-PCB-9MM
- J1: value (none) -> SERVO 1
- J2: value (none) -> SERVO 2
- moved S2 485.6 mm to (98.4, 37.1), turned to 180 degrees
- moved I2C-0 456.4 mm to (12.7, 72.4), turned to 180 degrees
- moved R16 407.2 mm to (16.4, 31.8)
- moved R15 395.4 mm to (16.4, 36.8)
- moved LED16 394.8 mm to (10.2, 31.8), turned to 180 degrees
- moved J2 394.3 mm to (223.5, 72.4), turned to 180 degrees
- moved LED15 386.1 mm to (10.2, 36.8), turned to 180 degrees
- moved R14 384.9 mm to (16.5, 41.9)
- moved U3 375.7 mm to (188.0, 57.1)
- moved LED14 372.4 mm to (10.2, 41.9), turned to 180 degrees
- moved R13 371.3 mm to (16.6, 47.0)
- moved LED13 358.7 mm to (10.2, 47.0), turned to 180 degrees
- moved IC2 358.2 mm to (151.1, 8.89)
- moved J1 357.3 mm to (210.8, 72.4), turned to 180 degrees
- moved IC1 315.7 mm to (105.4, 8.89)
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Connections:
- removed net KNOB1: KNOB1.P$2
- removed net VCC: KNOB1.P$3
- new net N$10: R4.1, S4.A
- new net N$15: R9.1, S9.A
- new net N$16: R10.1, S10.A
- new net N$17: R11.1, S11.A
- new net N$18: R12.1, S12.A
- new net N$19: R17.1, S13.A
- new net N$20: R18.1, S14.A
- new net N$21: R19.1, S15.A
- new net N$22: R20.1, S16.A
- new net N$8: R2.1, S2.A
- new net N$9: R3.1, S3.A
- net +5V: now also R5.1, R6.1, REG1.IN+, TM1.1, TM10.1, TM11.1, TM12.1, TM13.1, TM14.1, TM15.1, TM16.1, TM2.1, TM3.1, TM4.1, TM9.1; no longer J_REG_5V_1.VIN
- net A1: now also TM1.2, U$1.14; no longer U$1.33
- net A10: now also TM10.2, U$1.DAC1; no longer U$1.14
- net A11: now also TM11.2, U$1.A10; no longer U$1.15
- net A12: now also TM12.2, U$1.A11; no longer U$1.16
- net A2: now also TM2.2, U$1.15; no longer U$1.34
- net A3: now also TM3.2, U$1.16; no longer U$1.35
- net A4: now also TM4.2, U$1.33; no longer U$1.36
- net A5: now also TM13.2, U$1.34; no longer U$1.39
- net A6: now also TM14.2, U$1.35; no longer U$1.DAC0
- net A7: now also TM15.2, U$1.36; no longer U$1.DAC1
- net A8: now also TM16.2, U$1.39; no longer U$1.A10
- net A9: now also TM9.2, U$1.DAC0; no longer U$1.A11
- net AGND: now also TM1.3, TM10.3, TM11.3, TM12.3, TM13.3, TM14.3, TM15.3, TM16.3, TM2.3, TM3.3, TM4.3, TM9.3; no longer KNOB1.P$1
- net B1: now also S1.3; no longer BUTTON1.3
- net B10: now also S10.3
- net B11: now also S11.3
- net B12: now also S12.3
- net B2: now also S2.3
- net B3: now also S3.3
- net B4: now also S4.3
- net B5: now also S13.3
- net B6: now also S14.3
- net B7: now also S15.3
- net B8: now also S16.3
- net B9: now also S9.3
- net GND: now also REG1.IN-, REG1.OUT-, S1.1, S1.C, S10.1, S10.C, S11.1, S11.C, S12.1, S12.C, S13.1, S13.C, S14.1, S14.C, S15.1, S15.C, S16.1, S16.C, S2.1, S2.C, S3.1, S3.C, S4.1, S4.C, S9.1, S9.C; no longer BUTTON1.1, J_REG_5V_1.GND, LED1.K
- net I2C_SCL: now also R5.2
- net I2C_SDA: now also R6.2
- net LED10: now also R10.2
- net LED11: now also R11.2
- net LED12: now also R12.2
- net LED2: now also R2.2
- net LED3: now also R3.2
- net LED4: now also R4.2
- net LED5: now also R17.2
- net LED6: now also R18.2
- net LED7: now also R19.2
- net LED8: now also R20.2
- net LED9: now also R9.2
- net N$1: now also S1.A; no longer LED1.A
- net S1: no longer J2.3
- net S2: now also J2.3
- net VMOT: now also REG1.OUT+; no longer J_REG_5V_1.VOUT
Routing:
- added copper zone on layer 16, net GND
- added copper zone on layer 1, net N$11
