File: PCBs/MOL-v1.brd (EAGLE design)
At the start: 252.7 x 75.9 mm, 27 parts, among them IC1 ULN2803, IC2 ULN2803, U1 SN74LVC2G04DBV, U2 JOYSTICKPTH, U3 JOYSTICKPTH

Commit message: using git for real
Parts:
- removed BUTTON1: DTS-6, switch-tact:DTS-6
- removed J_REG_5V_1: POLOLU_VOLTAGE_REGULATORS_3PIN, CMU-ArtFab:POLOLU_5V-12V_STEPUP_U3V12F5-U3V12F12
- removed KNOB1: (no value), CMU-ArtFab:ALPS_POT
- removed LED1: (no value), led:LED3MM
- added GND-SHRT, VIN, VOUT: (no value), CMU-ArtFab:1X02_LOCK
- added R10, R11, R12, R17, R18, R19, R2, R20, R3, R4, R5, R6, R9: (no value), SparkFun-Resistors:AXIAL-0.3EZ
- added S10, S11, S12, S3, S4, S5, S6, S7, S8, S9: SW-LEDPTH, Daniel:TR2-SWITCH-MOMENTARY-LED
- added TM1, TM10, TM11, TM12, TM2, TM3, TM4, TM5, TM6, TM7, TM8, TM9: (no value), Daniel:TRIM-PCB-9MM
- J1: value (none) -> SERVO 1
- J2: value (none) -> SERVO 2
- R1, R13, R14, R15, R16: device CMU-ArtFab:R0603 -> SparkFun-Resistors:AXIAL-0.3EZ
- moved S2 476.8 mm to (58.0, 39.8), turned to 180 degrees
- moved I2C-0 424.8 mm to (129.5, 2.54), flipped to the bottom
- moved R16 405.5 mm to (26.9, 27.7), flipped to the bottom, turned to 270 degrees
- moved LED16 401.8 mm to (26.9, 35.4), turned to 270 degrees
- moved R15 387.4 mm to (21.8, 27.7), flipped to the bottom, turned to 270 degrees
- moved LED15 387.0 mm to (21.8, 35.4), turned to 270 degrees
- moved R14 371.0 mm to (16.6, 27.7), flipped to the bottom, turned to 270 degrees
- moved LED14 367.3 mm to (16.8, 35.4), turned to 270 degrees
- moved IC2 352.6 mm to (130.8, 15.2), flipped to the bottom
- moved U3 351.6 mm to (143.5, 59.7)
- moved R13 351.4 mm to (11.8, 27.7), flipped to the bottom, turned to 270 degrees
- moved LED13 347.6 mm to (11.7, 35.4), turned to 270 degrees
- moved J2 331.0 mm to (162.6, 43.2), turned to 90 degrees
- moved IC1 320.6 mm to (104.1, 15.2), flipped to the bottom
- moved J1 308.1 mm to (162.6, 52.1), turned to 90 degrees
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Connections:
- removed net KNOB1: KNOB1.P$2
- removed net VCC: KNOB1.P$3
- new net N$10: R4.P$1, S4.A
- new net N$15: R9.P$1, S9.A
- new net N$16: R10.P$1, S10.A
- new net N$17: R11.P$1, S11.A
- new net N$18: R12.P$1, S12.A
- new net N$19: R17.P$1, S5.A
- new net N$20: R18.P$1, S6.A
- new net N$21: R19.P$1, S7.A
- new net N$22: R20.P$1, S8.A
- new net N$8: R2.P$1, S2.A
- new net N$9: R3.P$1, S3.A
- net +3V3: now also TM1.1, TM10.1, TM11.1, TM12.1, TM2.1, TM3.1, TM4.1, TM5.1, TM6.1, TM7.1, TM8.1, TM9.1
- net +5V: now also R5.P$1, R6.P$1, VIN.1; no longer J_REG_5V_1.VIN
- net A1: now also TM1.2, U$1.14; no longer U$1.33
- net A10: now also TM10.2, U$1.DAC1; no longer U$1.14
- net A11: now also TM11.2, U$1.A10; no longer U$1.15
- net A12: now also TM12.2, U$1.A11; no longer U$1.16
- net A2: now also TM2.2, U$1.15; no longer U$1.34
- net A3: now also TM3.2, U$1.16; no longer U$1.35
- net A4: now also TM4.2, U$1.33; no longer U$1.36
- net A5: now also TM5.2, U$1.34; no longer U$1.39
- net A6: now also TM6.2, U$1.35; no longer U$1.DAC0
- net A7: now also TM7.2, U$1.36; no longer U$1.DAC1
- net A8: now also TM8.2, U$1.39; no longer U$1.A10
- net A9: now also TM9.2, U$1.DAC0; no longer U$1.A11
- net AGND: now also TM1.3, TM10.3, TM11.3, TM12.3, TM2.3, TM3.3, TM4.3, TM5.3, TM6.3, TM7.3, TM8.3, TM9.3; no longer KNOB1.P$1
- net B1: now also S1.3; no longer BUTTON1.3
- net B10: now also S10.3
- net B11: now also S11.3
- net B12: now also S12.3
- net B2: now also S2.3
- net B3: now also S3.3
- net B4: now also S4.3
- net B5: now also S5.3
- net B6: now also S6.3
- net B7: now also S7.3
- net B8: now also S8.3
- net B9: now also S9.3
- net GND: now also GND-SHRT.2, S1.1, S1.C, S10.1, S10.C, S11.1, S11.C, S12.1, S12.C, S2.1, S2.C, S3.1, S3.C, S4.1, S4.C, S5.1, S5.C, S6.1, S6.C, S7.1, S7.C, S8.1, S8.C, S9.1, S9.C, VIN.2, VOUT.1; no longer BUTTON1.1, J_REG_5V_1.GND, LED1.K
- net GND_MOT: now also GND-SHRT.1
- net I2C_SCL: now also R5.P$2
- net I2C_SDA: now also R6.P$2
- net LED1: now also R1.P$2; no longer R1.2
- net LED10: now also R10.P$2
- net LED11: now also R11.P$2
- net LED12: now also R12.P$2
- net LED2: now also R2.P$2
- net LED3: now also R3.P$2
- net LED4: now also R4.P$2
- net LED5: now also R17.P$2
- net LED6: now also R18.P$2
- net LED7: now also R19.P$2
- net LED8: now also R20.P$2
- net LED9: now also R9.P$2
- net N$1: now also R1.P$1, S1.A; no longer LED1.A, R1.1
- net N$2: now also R13.P$1; no longer R13.1
- net N$3: now also R14.P$1; no longer R14.1
- net N$4: now also R15.P$1; no longer R15.1
- net N$7: now also R16.P$1; no longer R16.1
- net S1: no longer J2.3
- net S2: now also J2.3
- net U1: now also R13.P$2; no longer R13.2
- net U2: now also R14.P$2; no longer R14.2
- net U3: now also R15.P$2; no longer R15.2
- net U4: now also R16.P$2; no longer R16.2
- net VMOT: now also VOUT.2; no longer J_REG_5V_1.VOUT
Routing:
- net GND: track 0.00 -> 483.1 mm
- net +3V3: track 0.00 -> 457.0 mm, vias 0 -> 1
- net AGND: track 0.00 -> 342.2 mm
- net S_JOYH: track 0.00 -> 200.7 mm, vias 0 -> 2
- net S2: track 0.00 -> 187.8 mm
- net S_JOYB: track 0.00 -> 176.2 mm
- net S_JOYV: track 0.00 -> 170.8 mm, vias 0 -> 1
- net M_PWMA: track 0.00 -> 164.0 mm, vias 0 -> 2
- net L1: track 0.00 -> 163.9 mm, vias 0 -> 1
- net S1: track 0.00 -> 155.2 mm, vias 0 -> 1
- net +5V: track 0.00 -> 144.0 mm, vias 0 -> 3
- net M_PWMB: track 0.00 -> 141.7 mm, vias 0 -> 4
- net A12: track 0.00 -> 140.8 mm, vias 0 -> 3
- net M_AIN: track 0.00 -> 136.0 mm, vias 0 -> 1
- net A10: track 0.00 -> 135.5 mm, vias 0 -> 3
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Other:
- board size 252.7 x 75.9 mm -> 165.1 x 77.1 mm
