File: PCBs/MOL-v1.brd (EAGLE design)
At the start: 165.1 x 77.1 mm, 61 parts, among them IC1 ULN2803, IC2 ULN2803, J1 SERVO 1, J2 SERVO 2, U1 SN74LVC2G04DBV, U2 JOYSTICKPTH, U3 JOYSTICKPTH

Commit message: breakouts
Parts:
- added J3, J4, J5, J6, J7, J8: (no value), SparkFun-Connectors:1X03_NO_SILK
- J1, J2: device SparkFun-Connectors:1X03_LOCK -> SparkFun-Connectors:1X03_LOCK@1
Connections:
- net +3V3: now also J3.1, J4.1, J5.1, J6.1, J7.1, J8.1
- net A1: now also J3.2
- net A10: now also J8.2
- net A2: now also J4.2
- net A5: now also J5.2
- net A6: now also J6.2
- net A9: now also J7.2
- net AGND: now also J3.3, J4.3, J5.3, J6.3, J7.3, J8.3
Routing:
- net AGND: track 342.2 -> 436.8 mm, vias 0 -> 1
- net +3V3: track 457.0 -> 507.7 mm, vias 1 -> 0
- net A2: track 79.6 -> 113.0 mm, vias 1 -> 0
- net S_JOYH: track 200.7 -> 171.0 mm, vias 2 -> 3
- net A1: track 68.1 -> 95.0 mm
- net S2: track 187.8 -> 161.0 mm, vias 0 -> 1
- net L4: track 107.5 -> 133.1 mm
- net L1: track 163.9 -> 139.1 mm
- net A9: track 127.1 -> 150.3 mm, vias 3 -> 2
- net GND: track 483.1 -> 463.0 mm
- net A10: track 135.5 -> 155.0 mm
- net LED1: track 71.3 -> 89.5 mm
- net A8: track 93.4 -> 110.3 mm, vias 3 -> 2
- net A6: track 91.7 -> 107.5 mm, vias 4 -> 3
- net S_JOYV: track 170.8 -> 186.4 mm
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Other:
- board size 165.1 x 77.1 mm -> 165.1 x 81 mm
- board text removed: "***The TEENSY is on the BOTTOM side of the board; KNOBS and BUTTONS are on the TOP side of the board."

Commit message: sent to fab
Routing:
- net M_BIN: track 124.1 -> 204.6 mm, vias 2 -> 0
- net M_PWMA: track 159.8 -> 228.5 mm, vias 1 -> 2
- net L2: track 116.4 -> 180.1 mm, vias 2 -> 1
- net M_PWMB: track 137.5 -> 198.6 mm, vias 2 -> 3
- net L1: track 139.1 -> 200.1 mm, vias 1 -> 2
- net L6: track 99.0 -> 148.2 mm
- net L4: track 133.1 -> 178.2 mm, vias 1 -> 2
- net L7: track 96.1 -> 140.1 mm
- net L5: track 100.8 -> 143.4 mm
- net S1: track 168.1 -> 210.7 mm, vias 2 -> 0
- net +3V3: track 507.7 -> 549.5 mm
- net LED1: track 89.5 -> 59.6 mm, vias 0 -> 2
- net M_AIN: track 137.8 -> 166.0 mm, vias 1 -> 5
- net A8: track 110.3 -> 86.2 mm, vias 2 -> 3
- net S_JOYV: track 186.4 -> 163.3 mm, vias 1 -> 3
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